File: electronics/test-article/thermabrick-test-article.kicad_sch (KiCad schematic)
At the start: 29 parts, among them J1 NEMA 5-15P cord, 14/3 SJT, K1 30 A DPDT, 120 VAC coil, M1 12 V blower, SW1 STOP (NC), SW2 START (NO), U1 SSR-25DA zero-cross, U10 MAX6675 module, U2 REX-C100, relay out, K input, U3 Buck 12 V to 5 V, 3 A, U4 Logic-level MOSFET PWM module, U5 ESP32 DevKit (ESP32-WROOM-32), U6 MAX6675 module, U7 MAX6675 module, U8 MAX6675 module, U9 MAX6675 module

Commit message: Add controller enclosure model TBK-DWG-005 Rev P1
- cad/src/enclosure.py: parametric 250 x 200 x 150 mm enclosure with
  DIN rail, supply, relay, SSR heat sink, controller, REX-C100,
  buttons and glands; fit check (3 mm clearance, lid closure) that
  also shows the original 100 mm deep box fails; STEP and STL
- cad/src/sheets.py: TBK-DWG-005 sheet, per-sheet iso options
- TBK-DWG-003 Rev P2: PS1 is a DIN-rail HDR-15-12 12 V 1.25 A supply
- BOM: enclosure, supply, DIN rail, glands, lever connectors and
  earth stud corrected; test article now $635.70, over $600
- TBK-PRC-002 v0.7, TBK-REQ-001 v0.5, TBK-PRB-001 v0.4, README and
  BOM notes updated with the overrun and options; PDFs re-rendered

Co-Authored-By: Claude Opus 5.5 <noreply@anthropic.com>
Parts:
- PS1: value 12 V 5 A -> HDR-15-12, 12 V 1.25 A
Other:
- note added: "9. PS1 and K1 mount on the DIN rail; layout in enclosure drawing TBK-DWG-005."
Changed lines of the file:
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@@
     (title "ThermaBrick test article controller")
     (date "2026-09-24")
-    (rev "P1")
+    (rev "P2")
     (company "Open Hardware Portfolio, amishchadha.com")
     (comment 1 "TBK-DWG-003. Generated by electronics/src/schematic.py; do not edit by hand.")
@@
       )
     )
-    (property "Value" "12 V 5 A"
+    (property "Value" "HDR-15-12, 12 V 1.25 A"
       (at 25.4 152.4 0)
       (effects
@@
     (effects
       (font
+        (size 1.27 1.27)
+      )
+      (justify left bottom)
+    )
+  )
+  (text "9. PS1 and K1 mount on the DIN rail; layout in enclosure drawing TBK-DWG-005."
+    (exclude_from_sim no)
+    (at 254 59.69 0)
+    (effects
+      (font
