File: archive/out-of-phase-trl4/electronics/controller-board/thermabrick-controller-board.kicad_sch (KiCad schematic)
At the start: 19 parts, among them J1 12 V in, J2 SSR drive, J3 Blower, Q1 2N3904, Q2 IRLZ44N, U1 R-78E5.0-1.0, U2 ESP32-DevKitC V4, U3 MAX6675 module, T1 well wall, U4 MAX6675 module, T3 sand center, U5 MAX6675 module, T4 sand outer, U6 MAX6675 module, T5 outlet air, U7 MAX6675 module, T6 room air

Commit message: Accept all recommendations (DDR-002), switch footer to designmolecule.com, add README write-up with new inspiration point
Co-Authored-By: Claude Opus 5.5 <noreply@anthropic.com>
Claude-Session: https://claude.ai/code/session_01XuhhSU4W6fYhgCfURbrkut
Other:
- company: Open Hardware Portfolio, amishchadha.com -> Open Hardware Portfolio, designmolecule.com
Changed lines of the file:
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@@
     (date "2026-09-24")
     (rev "P1")
-    (company "Open Hardware Portfolio, amishchadha.com")
+    (company "Open Hardware Portfolio, designmolecule.com")
     (comment 1 "TBK-DWG-004 schematic. Generated by electronics/src/board.py; do not edit by hand.")
     (comment 2 "Licensed CERN-OHL-S-2.0")
