File: archive/out-of-phase-trl4/electronics/test-article/thermabrick-test-article.kicad_sch (KiCad schematic)
At the start: 29 parts, among them J1 NEMA 5-15P cord, 14/3 SJT, K1 30 A DPDT, 120 VAC coil, M1 12 V blower, SW1 STOP (NC), SW2 START (NO), U1 SSR-25DA zero-cross, U10 MAX6675 module, U2 REX-C100, relay out, K input, U3 Buck 12 V to 5 V, 3 A, U4 Logic-level MOSFET PWM module, U5 ESP32 DevKit (ESP32-WROOM-32), U6 MAX6675 module, U7 MAX6675 module, U8 MAX6675 module, U9 MAX6675 module

Commit message: Accept all recommendations (DDR-002), switch footer to designmolecule.com, add README write-up with new inspiration point
Co-Authored-By: Claude Opus 5.5 <noreply@anthropic.com>
Claude-Session: https://claude.ai/code/session_01XuhhSU4W6fYhgCfURbrkut
Other:
- company: Open Hardware Portfolio, amishchadha.com -> Open Hardware Portfolio, designmolecule.com
Changed lines of the file:
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@@
     (date "2026-09-24")
     (rev "P2")
-    (company "Open Hardware Portfolio, amishchadha.com")
+    (company "Open Hardware Portfolio, designmolecule.com")
     (comment 1 "TBK-DWG-003. Generated by electronics/src/schematic.py; do not edit by hand.")
     (comment 2 "Licensed CERN-OHL-S-2.0")
